Commit message: Implement Phase 1: simulation model update for Jetson modification
Complete all 6 Phase 1 tasks to update the simulation model for the
Jetson Orin Nano replacement of the Raspberry Pi Zero 2W.

Task 1.1 — Mass and inertia calculations:
- trunk_assembly: 698.5g → 1024.5g (+Jetson 176g, +batteries 90g,
  +DC-DC 15g, +thermal partition 37g, +wiring 8g)
- head_assembly: 352.6g → 342.6g (-Pi Zero 10g)
- Total robot: 2061.5g → 2377.5g (+15.3%)
- Full derivation in docs/jetson-mod/mass_inertia_calculations.md

Task 1.2 — Placeholder STL meshes:
- jetson_orin_nano.stl (103x90.5x34.77mm box, meters)
- thermal_partition.stl (3x110x90mm thin slab, meters)
- dcdc_converter.stl (43x21x14mm box, meters)

Task 1.3 — robot_motors.xml updated:
- Replaced raspberrypizerow mesh with jetson_orin_nano, thermal_partition,
  dcdc_converter meshes
- Added Jetson/partition/DC-DC geoms in trunk_assembly (contype=0)
- Removed Pi Zero geom from head_assembly
- Updated trunk and head inertial properties

Task 1.4 — robot.xml updated with same changes as Task 1.3

Task 1.5 — robot.urdf updated:
- Removed Pi Zero visual/collision from head_assembly
- Added Jetson/partition/DC-DC visual/collision to trunk_assembly
- Updated inertial elements for both bodies

Task 1.6 — Test infrastructure:
- pytest.ini with phase markers
- tests/conftest.py with shared fixtures
- tests/test_mass_inertia.py (6 tests)
- tests/test_model_integrity.py (24 tests)
- All 30 tests pass, 5000-step stability verified

Co-Authored-By: Claude Opus 4.6 (1M context) <noreply@anthropic.com>

File: mini_bdx/robots/open_duck_mini_v2/robot.urdf (robot description, URDF)
Before this commit: robot onshape, 21 links, 20 joints
Links:
- link head_assembly: mass 0.35258298534369564292 -> 0.342583; geometry collision mesh filename=package:///board.stl; collision mesh filename=package:///drive_palonier.stl
- link trunk_assembly: mass 0.69852641931996084512 -> 1.024526; geometry collision mesh filename=package:///battery_pack_lid.stl; collision mesh filename=package:///bms.stl

Commit message: Implement Phase 2 (Tasks 2.1-2.3) and migrate servos from STS3215 to STS3250
Phase 2 Implementation:
- Task 2.1: MJCF→USD conversion script with MJCF importer extension fix
- Task 2.2: ArticulationCfg with BAM-identified STS3250 motor parameters
- Task 2.3: Isaac Lab locomotion env (DuckRewards, PPO config, Gym registration)

STS3215 → STS3250 Servo Migration:
- Upgrade all 14 servos to Feetech STS3250 (50 kg.cm stall, 74.5g, 12V)
- BAM parameters from kscalelabs/sysid id008: kp=45.53, kd=1.346,
  armature=0.040, friction=0.200, effort_limit=8.716 Nm
- Updated MJCF/URDF/USD model masses (+19.5g per servo, +95g battery/BMS)
- Battery: 2S2P 7.4V → 3S2P 11.1V (6x 18650 cells)
- New total robot mass: 2.746 kg (was 2.378 kg)
- Robot now holds Z=0.195m under gravity (was 0.052m with STS3215)

Verification: 53/53 pytest + 10/10 Isaac Sim checks pass.

Co-Authored-By: Claude Opus 4.6 (1M context) <noreply@anthropic.com>

File: mini_bdx/robots/open_duck_mini_v2/robot.urdf (robot description, URDF)
Before this commit: robot onshape, 21 links, 20 joints
Links:
- link head_assembly: mass 0.342583 -> 0.362083
- link hip_roll_assembly: mass 0.06648000000000005294 -> 0.08598000000000005294
- link hip_roll_assembly_2: mass 0.06648000000000005294 -> 0.08598000000000005294
- link knee_and_ankle_assembly: mass 0.12407000000000001361 -> 0.14357000000000001361
- link knee_and_ankle_assembly_2: mass 0.072590000000000057256 -> 0.092090000000000057256
- link knee_and_ankle_assembly_3: mass 0.12407000000000001361 -> 0.14357000000000001361
- link knee_and_ankle_assembly_4: mass 0.072590000000000057256 -> 0.092090000000000057256
- link left_roll_to_pitch_assembly: mass 0.075160000000000060094 -> 0.094660000000000060094
- link neck_pitch_assembly: mass 0.066180000000000058225 -> 0.085680000000000058225
- link neck_yaw_assembly: mass 0.09180988857925044544 -> 0.11130988857925044544
- link right_roll_to_pitch_assembly: mass 0.075160000000000060094 -> 0.094660000000000060094
- link trunk_assembly: mass 1.024526 -> 1.178026

Commit message: Part 2: chassis/shell CAD modifications (spine cut, vents, hump extension)
Applies the layout v2.1 cut list to the actual meshes via a reproducible
pipeline (scripts/generate_cad_mods.py, trimesh + manifold3d booleans).
Every modified part verified watertight and single-component; sim meshes
(meters) and print/ copies (mm) both regenerated.

- trunk_bottom: central spine removed (SPINE_CUT_BOX; -60.3 cm^3) — the
  Jetson bay is now physically clear; trunk_top mid-span load flows
  through the hip-yaw towers. Regression test tightened from
  box-allowance to ZERO Jetson<->trunk_bottom intrusion.
- body_middle_bottom: +y port opening x[-80,-54] z[-15,24] (the only
  walled section of the Jetson I/O edge), 3x -y exhaust louvers at fin
  height, 4x D8 floor bosses topping 0.1 mm under the Jetson base plate
  (flat seats + pilot bases; no vendor hole pattern exists for P3768).
- body_front: 6 inlet slots (20x6) at plenum height feeding the fan
  intake above the heatsink.
- body_back: battery hump extended rearward (outer to x=-170, bore
  y +/-20.5 sparing the USB-C charger mount) so the 6-cell 3S2P pack
  fits (2 front + 2x2 rear grid).
- NEW print/thermal_partition.stl: 2 mm PLA wall with 45-deg bottom
  corner chamfers and 8x5 cable notch (mica sheet is purchased).

Physics: measured boolean volume deltas booked into the inertial
generator at their delta centroids (printed-PLA effective density
1.116 g/cm^3 = 0.9x solid, documented): trunk -89.4 g -> 1.088626 kg,
total robot 2.656149 kg (MuJoCo-verified). fullinertia updated in all
three model files; fixtures + hardware-specs + CLAUDE.md + layout doc
updated. Standing CoM -6.3 mm aft of foot origins (measured).

Tests: 88/88 pass, including the tightened zero-intrusion spine test
and the mesh-level relocated-component checks.

Co-Authored-By: Claude Fable 5 <noreply@anthropic.com>

File: mini_bdx/robots/open_duck_mini_v2/robot.urdf (robot description, URDF)
Before this commit: robot onshape, 21 links, 20 joints
Links:
- link trunk_assembly: mass 1.178026 -> 1.088626

Commit message: Part 2 review fixes: verified partition fit, port mullion, exact delta tensors
The adversarial review of e7bf790 (3 verifiers: mesh geometry, physics
booking, design/structure) approved the physics bookkeeping bit-exact but
found four design defects. All fixed:

- Printed partition could not seat: the 45-deg corner chamfers (16.97 mm
  legs, not the commented 12 — sqrt-2 error) did not clear the shell wall
  fillets (measured slope 24.6 deg), leaving 73.7 mm^3 interference; a
  first fix attempt left 271 then 11 mm^3 (floor ridge wider/taller than
  sampled). Corners now cut to the measured fillet profile plus a 1 mm
  bottom rabbet over the ridge, and generate_cad_mods.py ASSERTS an
  exact-boolean zero-interference fit of the posed printed part against
  body_middle_bottom/trunk_bottom/trunk_top on every run (now 0.00 mm^3).
- Port opening merged with the leg cutout (its true edge is x=-54.5, not
  -50) and left a 0.2-1.6 mm sill knife-edge: shrunk to x[-80,-58]
  (3.5 mm mullion), floor dropped to z=-16.5; louvers reduced to 2 (the
  third had merged with the cutout).
- Shell deltas were point/box-booked (~1% Iyy/Izz bias): the generator now
  emits exact signed tensors per removed/added diff solid to
  scripts/cad_mod_deltas.json, which compute_trunk_inertial.py loads —
  closing the mesh->physics pipeline. Generator is also idempotent now
  (restores pristine meshes from BASELINE_COMMIT adbc082 each run).
- Ribs/tray honesty: measured spine-to-trunk_top contact was 2.2 mm^3
  (never real support) — documented with the no-ribs justification;
  Jetson retention tray, 6-cell lid + rear-cell cradle, and partition
  rails are now EXPLICIT open deferrals (with WiFi-antenna drill warning).
- Extra cells seated on the bore floor (z 0.0325 -> 0.0306); density
  uncertainty band (+/-10-30 g on the bulky spine) documented; stale
  mass_inertia_calculations notice + ledger comment updated.

New model values (MuJoCo-verified): trunk 1.089544 kg, total 2.657067 kg,
fullinertia per compute_trunk_inertial.py output; fixtures + hardware-specs
+ layout doc synced. Tests: 88/88 pass.

Co-Authored-By: Claude Fable 5 <noreply@anthropic.com>

File: mini_bdx/robots/open_duck_mini_v2/robot.urdf (robot description, URDF)
Before this commit: robot onshape, 21 links, 20 joints
Links:
- link trunk_assembly: mass 1.088626 -> 1.089544

Commit message: fix(urdf): repair robot.urdf to zero validator errors — Task M7 branch A
robot.urdf was an onshape-to-robot export that had never validated: 244
blocking findings. It is not in any training or evaluation code path (the USD
comes from robot_motors.xml), but it is the standard interchange format and, as
this change shows, a genuinely useful independent check on the MJCF.

Repairs:

  266 mesh references were `package:///<name>.stl` — a package:// URI with an
  EMPTY package name, which no consumer can resolve. Rewritten to plain paths
  relative to the URDF; all 47 distinct meshes verified present on disk first.

  The four frame links (trunk, left_foot, right_foot, head) carried
  zero-diagonal inertia tensors, which are not legal for a rigid body. They are
  pure kinematic frames attached by fixed joints, so the <inertial> is REMOVED
  rather than replaced with an invented epsilon — the urdf skill explicitly
  endorses frame-only links omitting mass and geometry. These are the same four
  markers the MJCF declares at mass=1e-09 (known_issues.md PLANT-1b).

  A design ledger now heads the file, per the urdf skill's contract: units,
  frame semantics, topology, the repairs applied, the deliberate <mujoco> /
  <joint_properties> extensions that are NOT to be "fixed", and an explicit
  statement that the inertia tensors are inherited from the Onshape export and
  are not certified here — Phase M will make them stale.

Validator now reports 0 errors:

  OK robot 'onshape', root 'trunk_assembly', 21 links, 20 joints (16 movable),
     266 resolved mesh references, total mass 2.657 kg

That total mass independently corroborates the MJCF's 2.657067 kg — two
descriptions from different toolchains agreeing on the plant. The URDF also
renders now; it previously failed with "No link mesh loaded for robot".

Adds tests/test_urdf_consistency.py (7 tests) so the two descriptions cannot
drift again. It PARSES both files rather than grepping source text, because
this repo already has a suite that greps and lets 5 of 7 seeded regressions
through (TEST-1). It compares movable joint names, joint parent/child topology,
the body/link set, the root link and that it carries real mass, total mass, and
that every mesh reference resolves. It deliberately does NOT compare inertia
tensors or joint limits, which are provisional until Phase M lands.

Mutation-tested, because a test that cannot fail is worse than no test. Five
mutations, each caught by exactly one assertion, all reverted:
  rename a joint in the URDF only            -> joint-name test fails
  restore one package:/// URI                 -> mesh-resolution test fails
  rewire a joint's parent                     -> topology test fails
  point a mesh at a nonexistent file          -> mesh-resolution test fails
  delete a link                               -> link-set test fails

Verified: pytest tests/ 110 passed (103 + 7 new); urdf validator 0 errors;
verify_known_issues.py 28/29 CONFIRMED, 0 REFUTED.

Co-Authored-By: Claude Opus 5 (1M context) <noreply@anthropic.com>

File: mini_bdx/robots/open_duck_mini_v2/robot.urdf (robot description, URDF)
Before this commit: robot onshape, 21 links, 20 joints
Links:
- link foot_assembly: geometry collision mesh filename=foot_bottom_pla.stl; collision mesh filename=foot_bottom_tpu.stl
- link foot_assembly_2: geometry collision mesh filename=foot_bottom_pla.stl; collision mesh filename=foot_bottom_tpu.stl
- link head: mass 1e-9 -> None
- link head_assembly: geometry collision mesh filename=board.stl; collision mesh filename=drive_palonier.stl
- link head_pitch_to_yaw: geometry collision mesh filename=head_pitch_to_yaw.stl; visual mesh filename=head_pitch_to_yaw.stl
- link hip_roll_assembly: geometry collision mesh filename=drive_palonier.stl; collision mesh filename=passive_palonier.stl
- link hip_roll_assembly_2: geometry collision mesh filename=drive_palonier.stl; collision mesh filename=passive_palonier.stl
- link knee_and_ankle_assembly: geometry collision mesh filename=drive_palonier.stl; collision mesh filename=left_cache.stl
- link knee_and_ankle_assembly_2: geometry collision mesh filename=drive_palonier.stl; collision mesh filename=left_knee_to_ankle_left_sheet.stl
- link knee_and_ankle_assembly_3: geometry collision mesh filename=drive_palonier.stl; collision mesh filename=left_knee_to_ankle_left_sheet.stl
- link knee_and_ankle_assembly_4: geometry collision mesh filename=drive_palonier.stl; collision mesh filename=left_knee_to_ankle_left_sheet.stl
- link left_antenna_holder: geometry collision mesh filename=antenna.stl; collision mesh filename=left_antenna_holder.stl
- link left_foot: mass 1e-9 -> None
- link left_roll_to_pitch_assembly: geometry collision mesh filename=drive_palonier.stl; collision mesh filename=left_roll_to_pitch.stl
- link neck_pitch_assembly: geometry collision mesh filename=drive_palonier.stl; collision mesh filename=neck_left_sheet.stl
- link neck_yaw_assembly: geometry collision mesh filename=drive_palonier.stl; collision mesh filename=head_yaw_to_roll.stl
- link right_antenna_holder: geometry collision mesh filename=antenna.stl; collision mesh filename=right_antenna_holder.stl
- link right_foot: mass 1e-9 -> None
- link right_roll_to_pitch_assembly: geometry collision mesh filename=drive_palonier.stl; collision mesh filename=passive_palonier.stl
- link trunk: mass 1e-9 -> None
- link trunk_assembly: geometry collision mesh filename=battery_pack_lid.stl; collision mesh filename=bms.stl

Commit message: feat(cad): six 18650s become real geometry, and the pack is proved to fit
Task M3. The robot is specified as 6x 18650 in 3S2P and compute_trunk_inertial.py
has always booked 180 g for the four "extra" cells -- but only TWO existed as
geometry. 180 g of the densest payload in the machine sat at a coordinate no
geometry occupied, and every clearance number was computed against a bay four
cells emptier than the build.

component_layout_v2.md gave the usable bore TWO different depths (28.4 mm in the
Layout table, 26.4 implied by cut-list item 4) and declared a 4-cell block that
overlapped each existing cell by ~11.9 cm3. New scripts/measure_battery_bay.py
ends that by measuring: 42 (x) x 41 (y) x 69 (z) mm. Every layout the plan lists
-- 3x2, 2x3, 6x1, 1x6 -- failed against it, best case 2384 mm3.

The hump is DEEPENED, not widened, and that reversed my first choice. Widening
looked cheaper until the measurement showed bms (y -28.5..-24.9) and
usb_c_charger (y -30.9..-25.7) hugging the old bore's -y wall with no obvious
home elsewhere in a trunk this full. Dodging them asymmetrically would offset
the 270 g pack +6.6 mm in y, about 0.65 mm of LATERAL CoM shift. Deepening keeps
the pack 2 wide, clears both untouched, stays laterally symmetric, and costs
~1.6 mm of AFT shift plus 23 mm of rear protrusion. Aft is the safer error:
sagittal shift is along the walking direction the gait already manages, while
lateral shift biases frontal-plane balance, which is the harder axis for a biped
and the one this policy falls on.

    bore x  -167..-125 (42 mm)  ->  -190..-123 (67 mm)
    bore y  ±20.5      (41 mm)  ->  ±22.0      (44 mm)
    outer x -170 mm             ->  -193 mm
    outer y ±24.0               ->  unchanged, so bms keeps its clearance

measure_battery_bay.py --from-mjcf now exits 0 with WORST = 0.00 mm3 -- better
than the shipped 2-cell layout, whose cells foul battery_pack_lid by 384.69 mm3
and whose holder fouls body_back by 513.67 mm3. Those pre-existing interferences
are recorded in docs/jetson-mod/battery_bay_before.txt so the acceptance bar is
honest about what the shipped robot has actually met.

Pack: 3 (x) x 2 (y) at 20.6 mm pitch centred (-156.5, 0, +32.5) mm. New
holder_6cell tray, 62.8 x 42.2 x 22 mm, Ø18.6 bores (a real wrapped 18650 is
18.3-18.6, not the nominal 18.0 the cell mesh models), 2.0 mm webs, watertight,
single-component, binary STL, byte-identical on re-run.

Two traps the plan did not name, both caught by measurement:
  - Sweeping CELLS alone found a 6 mm-wide "clear" band the 62.8 mm tray did not
    share. The tray has to be in the sweep. The final bore carries 4.2 mm of
    slack, because a 1 mm-wide window is a coincidence and not a clearance.
  - Sizing the tray as ROWS*PITCH + 2*WALL adds a full pitch of empty material at
    each end and gave 65.8 x 45.2 mm, which did not fit. It is sized to the
    cells: (ROWS-1)*PITCH + BORE + 2*WALL.

Deliberate deviation: the old 2-cell `holder` GEOM is removed rather than
"retained alongside" the new tray. A robot has one battery tray; keeping both
adds a phantom 7.5 cm3 part to the collision model and double-books it. The
holder mesh asset and holder.stl both remain for the 2-cell configuration. So
the unique (body, mesh, pose) count is 133 - 3 + 7 = 137, not the 140 the plan
predicted, and the test says so with the arithmetic.

Mass moved twice and both moves are booked. The deepened hump adds 25.44 g of
body_back shell, so the Part-2 CAD delta went from M2's -13.95 g to +0.38 g and
the trunk from 1.164076 to 1.178406 kg. The printed set is now 53 pieces /
1598.61 cm3 / 1199.50 g (was 52 / 1571.94 / 1163.14). part_mass_table.json,
cad_mod_deltas.json, print_process.json, print_guide.md and EXPECTED_PIECES were
all re-run or bumped here, not left to drift.

cells_extra_4x45g is KEPT with a TODO(M4), per the plan's branch for "M4 has not
landed": its position and tensor are corrected from the phantom
(-0.145, 0, 0.0306) / 38x38x65 to the measured (-0.1565, 0, 0.0325) /
59.2x38.6x65. A test asserts the marker exists while the lump does, so M4 cannot
silently double-book 180 g.

The USD is now stale by design. test_usd_not_stale and test_usd_meshes_not_stale
carry strict=True xfails naming Task M6, the Phase-M gate that regenerates it
once at the end rather than after every edit. NOTHING MAY TRAIN BEFORE M6:
Isaac Lab loads the USD, not the MJCF, so a stale USD trains on the old plant
silently.

tests/test_battery_pack.py: 12 tests. Suite 174 passed, 5 skipped, 3 xfailed.

Co-Authored-By: Claude Opus 5 (1M context) <noreply@anthropic.com>

File: mini_bdx/robots/open_duck_mini_v2/robot.urdf (robot description, URDF)
Before this commit: robot onshape, 21 links, 20 joints
Links:
- link trunk_assembly: geometry collision mesh filename=battery_pack_lid.stl; collision mesh filename=bms.stl
