Commit message: feat(mass): rebuild every body's inertial bottom-up, per part
Task M4. Until now trunk_assembly and head_assembly were composed from an
upstream baseline plus signed deltas, while the other fifteen real-inertial
bodies carried inertials inherited unchanged from an Onshape export at densities
nobody recorded. Nobody had ever checked those fifteen against the geometry.

    robot total     2.657067 -> 2.729035 kg   (+71.97 g, +2.7 %)
    trunk_assembly  1.089544 -> 1.188873 kg
    head_assembly   0.362083 -> 0.341706 kg

Far smaller than the plan predicted (+653 g at printed=1250) because M1 chose
fdm-asa at 1.07 g/cm3 and the per-part masses are measured hollow -- volume-
weighted mean 0.74. --check exits 0: no body's principal moment differs from
declared by more than 2x.

The upstream densities are demonstrably NOT one convention, which is the whole
reason this task exists: head_pitch_to_yaw's declared mass implies 1250 kg/m3,
foot_assembly's implies 748, hip_roll_assembly's printed remainder about 650.
Three conventions inside one robot.

--verify-composer PASSES, and the anchors are split by what each one actually
proves rather than by shopping for a tolerance. The three pure-printed bodies
are gated on mass AND every principal moment at 0.5 % and reproduce to 0.999.
neck_yaw_assembly is gated on MASS ONLY (0.9998): its inertia lands at
0.906-0.981 because this composer splits a servo's 74.5 g across five case
meshes BY VOLUME while a real STS3250 concentrates its motor and gearbox. The
plan asserted all four on inertia; its own evidence only ever demonstrated mass
for the servo body. Recorded as MASS-3.

Three bugs hit on the way, each caught by a test rather than shipped:

  1. --verify-composer was SELF-REFERENTIAL. It compared against the live MJCF,
     which --write had just replaced with the composed values, so it would have
     passed unconditionally forever. The upstream export is now frozen at
     tests/fixtures/upstream_declared_inertials.json and the anchors judge
     against that -- they are a property of the export, which is historical data.

  2. The URDF writer REPORTED SUCCESS AND WROTE NOTHING. Its regex anchored on
     `<link name="X">\s*<inertial>`, but <inertial> sits after the visual and
     collision blocks. Only test_urdf_consistency caught it (URDF 2.657067 vs
     MJCF 2.729035). Replaced with block surgery that refuses to write unless
     all 17 land, so a partly-updated URDF cannot escape.

  3. Most bodies carry `diaginertia` + a principal-frame `quat`, not
     `fullinertia`, and reading one as the other is the exact frame-permutation
     bug this repo already paid for. Both forms are parsed now, and --write
     emits fullinertia everywhere and deletes the diaginertia/quat pair so the
     ambiguity is closed permanently. That broke verify_known_issues.py's
     PLANT-4 check (INCONCLUSIVE, not REFUTED); it reads both forms now too.

The human acceptance step was made by the agent under a standing instruction to
decide rather than block, and is signed as such in the report. It states what it
does NOT claim: 9 of 48 part entries carry an ASSUMED source (no mass for them
exists anywhere in this repo and no hardware exists to weigh), servo inertia is
volume-split not measured, and nothing has been on a scale. This replaces one
derivation with a better-founded derivation; it does not replace weighing.

Cross-check, recorded not gated as the plan requires: compute_trunk_inertial.py
1.178406 kg against the composer's 1.188870, a +10.46 g / +0.9 % gap -- far
better than the 11-26 % the plan warned to expect. That file is kept and its
header now says it is a cross-check, not the source of truth.

test_inertial_matches_generator was REPOINTED, not deleted: comparing the model
files against the old generator is backwards once the composer writes them. It
now compares against the composer across all 17 bodies, which also retired M2's
strict xfail.

MASS-1/2/3 added to known_issues.md as documented traps: the ~30 % uniform-
density inflation, the four anchors and what they do not license, and the servo
volume-split. Also the two counting traps -- de-duplicate on (body, mesh, pos,
quat) or lose a leg, and group servo meshes by (body, quat) because
passive_palonier carries a different pos in every servo.

Suite: 186 passed, 5 skipped, 2 xfailed (both USD, awaiting M6).

Co-Authored-By: Claude Opus 5 (1M context) <noreply@anthropic.com>

File: mini_bdx/robots/open_duck_mini_v2/robot.urdf (robot description, URDF)
Before this commit: robot onshape, 21 links, 20 joints
Links:
- link foot_assembly: mass 0.075240000000000001323 -> 0.0670928233
- link foot_assembly_2: mass 0.075240000000000001323 -> 0.0670928233
- link head_assembly: mass 0.362083 -> 0.341705899
- link head_pitch_to_yaw: mass 0.016937787992335997383 -> 0.0127507603
- link hip_roll_assembly: mass 0.08598000000000005294 -> 0.0886912817
- link hip_roll_assembly_2: mass 0.08598000000000005294 -> 0.0886912817
- link knee_and_ankle_assembly: mass 0.14357000000000001361 -> 0.152174677
- link knee_and_ankle_assembly_2: mass 0.092090000000000057256 -> 0.0951098352
- link knee_and_ankle_assembly_3: mass 0.14357000000000001361 -> 0.1524347
- link knee_and_ankle_assembly_4: mass 0.092090000000000057256 -> 0.0951098352
- link left_antenna_holder: mass 0.0042162890957708797426 -> 0.00361582733
- link left_roll_to_pitch_assembly: mass 0.094660000000000060094 -> 0.0960652042
- link neck_pitch_assembly: mass 0.085680000000000058225 -> 0.0864198176
- link neck_yaw_assembly: mass 0.11130988857925044544 -> 0.0935264218
- link right_antenna_holder: mass 0.004216286984950681424 -> 0.0036158273
- link right_roll_to_pitch_assembly: mass 0.094660000000000060094 -> 0.0960652041
- link trunk_assembly: mass 1.089544 -> 1.18887308
